File: schematic/rfm_to_usb.sch (KiCad schematic (older format))
At the start: 16 parts, among them J1 USB_A, J2 ant, U1 STM32F103C8, U2 XC6206-33, X1 SWD_CON

Commit message: add uart, 2.8 mm lenght
Parts:
- removed J2: ant, Belkin_lib:pin_smd, symbol Connector:Conn_01x01
- added J2: Ant, Belkin_lib:pin_smd, symbol Connector_Generic:Conn_01x01
- added J3: UART_TX, Connector_PinSocket_2.54mm:PinSocket_1x01_P2.54mm_Vertical, symbol Connector_Generic:Conn_01x01
- added J4: UART_RX, Connector_PinSocket_2.54mm:PinSocket_1x01_P2.54mm_Vertical, symbol Connector_Generic:Conn_01x01
- added J5: GND, Connector_PinSocket_2.54mm:PinSocket_1x01_P2.54mm_Vertical, symbol Connector_Generic:Conn_01x01
- C1: symbol device:C -> Device:C
- C2, C3, C4, C5, C6: footprint Capacitor_SMD:C_0603_1608Metric -> Capacitor_SMD:C_0402_1005Metric; symbol device:C -> Device:C
- C7: footprint Capacitor_SMD:C_0805_2012Metric -> Capacitor_SMD:C_0402_1005Metric; symbol device:C -> Device:C
- R2, R3, R4: footprint Resistor_SMD:R_0603_1608Metric -> Resistor_SMD:R_0402_1005Metric; symbol device:R -> Device:R
- U1: footprint Package_QFP:TQFP-48_7x7mm_P0.5mm -> Belkin_lib:LQFP-48_7x7mm_Pitch0.5mm
- X1: footprint belkin:3WIRE_PADS -> Belkin_lib:SWD_CON
Connections:
- wire segments 111 -> 115
- no-connect marks 23 -> 21
Changed lines of the file:
@@
 encoding utf-8
 Sheet 1 1
-Title ""
+Title "RFM69 USB stick with UART input"
 Date "24 dec 2014"
 Rev ""
@@
 NoConn ~ 4500 4550
 NoConn ~ 4500 4450
-NoConn ~ 4500 4350
-NoConn ~ 4500 4250
 NoConn ~ 4500 4150
 NoConn ~ 4500 4050
@@
 NoConn ~ 4500 3500
 NoConn ~ 7500 3500
-NoConn ~ 7500 3400
+NoConn ~ 7500 3300
 NoConn ~ 7500 2900
 NoConn ~ 7500 2500
@@
 F 0 "X1" H 8500 4400 60  0000 C CNN
 F 1 "SWD_CON" H 8500 4800 60  0000 C CNN
-F 2 "belkin:3WIRE_PADS" H 8700 4600 60  0000 C CNN
+F 2 "Belkin_lib:SWD_CON" H 7850 4550 60  0001 C CNN
 F 3 "~" H 8700 4600 60  0000 C CNN
 	1    8700 4600
@@
 	3150 2750 3750 2750
 $Comp
-L device:R R2
+L Device:R R2
 U 1 1 6090FBC6
 P 7950 3600
 F 0 "R2" V 7850 3600 50  0000 C CNN
 F 1 "22R" V 7950 3600 50  0000 C CNN
-F 2 "Resistor_SMD:R_0603_1608Metric" V 7880 3600 50  0001 C CNN
+F 2 "Resistor_SMD:R_0402_1005Metric" V 7880 3600 50  0001 C CNN
 F 3 "" H 7950 3600 50  0001 C CNN
 	1    7950 3600
@@
 $EndComp
 $Comp
-L device:R R3
+L Device:R R3
 U 1 1 60910CC2
 P 7950 3700
 F 0 "R3" V 8050 3700 50  0000 C CNN
 F 1 "22R" V 7950 3700 50  0000 C CNN
-F 2 "Resistor_SMD:R_0603_1608Metric" V 7880 3700 50  0001 C CNN
+F 2 "Resistor_SMD:R_0402_1005Metric" V 7880 3700 50  0001 C CNN
 F 3 "" H 7950 3700 50  0001 C CNN
 	1    7950 3700
@@
 	7500 3700 7700 3700
 $Comp
-L device:R R4
+L Device:R R4
 U 1 1 60925512
 P 8300 3250
 F 0 "R4" V 8400 3250 50  0000 C CNN
 F 1 "1.5k" V 8300 3250 50  0000 C CNN
-F 2 "Resistor_SMD:R_0603_1608Metric" V 8230 3250 50  0001 C CNN
+F 2 "Resistor_SMD:R_0402_1005Metric" V 8230 3250 50  0001 C CNN
 F 3 "" H 8300 3250 50  0001 C CNN
 	1    8300 3250
@@
 	9400 1450 9600 1450
 $Comp
-L device:C C6
+L Device:C C6
 U 1 1 6065FC5F
 P 10850 1650
 F 0 "C6" H 10850 1750 50  0000 L CNN
 F 1 "0.1uF" H 10850 1550 50  0000 L CNN
-F 2 "Capacitor_SMD:C_0603_1608Metric" H 10888 1500 50  0001 C CNN
+F 2 "Capacitor_SMD:C_0402_1005Metric" H 10888 1500 50  0001 C CNN
 F 3 "" H 10850 1650 50  0001 C CNN
 	1    10850 1650
@@
 $EndComp
 $Comp
-L device:C C5
+L Device:C C5
 U 1 1 60661DD4
 P 10600 1650
 F 0 "C5" H 10600 1750 50  0000 L CNN
 F 1 "0.1uF" H 10600 1550 50  0000 L CNN
-F 2 "Capacitor_SMD:C_0603_1608Metric" H 10638 1500 50  0001 C CNN
+F 2 "Capacitor_SMD:C_0402_1005Metric" H 10638 1500 50  0001 C CNN
 F 3 "" H 10600 1650 50  0001 C CNN
 	1    10600 1650
@@
 $EndComp
 $Comp
-L device:C C4
+L Device:C C4
 U 1 1 60662044
 P 10350 1650
 F 0 "C4" H 10350 1750 50  0000 L CNN
 F 1 "0.1uF" H 10350 1550 50  0000 L CNN
-F 2 "Capacitor_SMD:C_0603_1608Metric" H 10388 1500 50  0001 C CNN
+F 2 "Capacitor_SMD:C_0402_1005Metric" H 10388 1500 50  0001 C CNN
 F 3 "" H 10350 1650 50  0001 C CNN
 	1    10350 1650
@@
 $EndComp
 $Comp
-L device:C C3
+L Device:C C3
 U 1 1 60662236
 P 9600 1650
 F 0 "C3" H 9400 1700 50  0000 L CNN
 F 1 "0.1uF" H 9300 1600 50  0000 L CNN
-F 2 "Capacitor_SMD:C_0603_1608Metric" H 9638 1500 50  0001 C CNN
+F 2 "Capacitor_SMD:C_0402_1005Metric" H 9638 1500 50  0001 C CNN
 F 3 "" H 9600 1650 50  0001 C CNN
 	1    9600 1650
@@
 $EndComp
 $Comp
-L device:C C2
+L Device:C C2
 U 1 1 60662563
 P 8600 1650
 F 0 "C2" H 8715 1696 50  0000 L CNN
 F 1 "0.1uF" H 8715 1605 50  0000 L CNN
-F 2 "Capacitor_SMD:C_0603_1608Metric" H 8638 1500 50  0001 C CNN
+F 2 "Capacitor_SMD:C_0402_1005Metric" H 8638 1500 50  0001 C CNN
 F 3 "" H 8600 1650 50  0001 C CNN
 	1    8600 1650
@@
 Wire Wire Line
 	10350 1800 10350 1850
-$Comp
-L Connector:Conn_01x01 J2
-U 1 1 6066C830
-P 3450 3200
-F 0 "J2" H 3600 3200 50  0000 C CNN
-F 1 "ant" H 3600 3150 50  0000 C CNN
-F 2 "Belkin_lib:pin_smd" H 3450 3200 50  0001 C CNN
-F 3 "~" H 3450 3200 50  0001 C CNN
-	1    3450 3200
-	1    0    0    1
-$EndComp
 Wire Wire Line
 	3250 3200 3150 3200
 $Comp
-L Belkin_lib:XC6206-33 U2
-U 1 1 60C0FB09
-P 9100 1450
-F 0 "U2" H 9100 1692 50  0000 C CNN
-F 1 "XC6206-33" H 9100 1601 50  0000 C CNN
-F 2 "Package_TO_SOT_SMD:SOT-23" H 9100 1650 50  0001 C CNN
-F 3 "" H 9200 1200 50  0001 C CNN
-	1    9100 1450
-	1    0    0    -1
-$EndComp
-$Comp
-L device:C C7
+L Device:C C7
 U 1 1 60C5E6EA
 P 9850 1650
 F 0 "C7" H 9965 1696 50  0000 L CNN
 F 1 "10uF" H 9965 1605 50  0000 L CNN
-F 2 "Capacitor_SMD:C_0805_2012Metric" H 9888 1500 50  0001 C CNN
+F 2 "Capacitor_SMD:C_0402_1005Metric" H 9888 1500 50  0001 C CNN
 F 3 "" H 9850 1650 50  0001 C CNN
 	1    9850 1650
@@
 $EndComp
 $Comp
-L device:C C1
+L Device:C C1
 U 1 1 60C5EB69
 P 8350 1650
@@
 F 0 "U1" H 4700 5450 50  0000 C CNN
 F 1 "STM32F103C8" H 7050 2150 50  0000 C CNN
-F 2 "Package_QFP:TQFP-48_7x7mm_P0.5mm" H 6000 3800 50  0000 C CNN
+F 2 "Belkin_lib:LQFP-48_7x7mm_Pitch0.5mm" H 4650 2150 50  0001 C CNN
 F 3 "" H 6000 3800 60  0000 C CNN
 	1    6000 3800
@@
 NoConn ~ 4500 2400
 Wire Wire Line
-	7700 3700 7700 3300
-Wire Wire Line
-	7700 3300 7500 3300
+	7700 3700 7700 3400
+Connection ~ 7700 3700
+Wire Wire Line
+	7700 3700 7800 3700
+$Comp
+L Connector_Generic:Conn_01x01 J2
+U 1 1 6224FE37
+P 3450 3200
+F 0 "J2" H 3400 3300 50  0000 L CNN
+F 1 "Ant" H 3400 3100 50  0000 L CNN
+F 2 "Belkin_lib:pin_smd" H 3450 3200 50  0001 C CNN
+F 3 "~" H 3450 3200 50  0001 C CNN
+	1    3450 3200
+	1    0    0    -1
+$EndComp
+$Comp
+L Belkin_lib:XC6206-33 U2
+U 1 1 62296064
+P 9100 1450
+F 0 "U2" H 9100 1692 50  0000 C CNN
+F 1 "XC6206-33" H 9100 1601 50  0000 C CNN
+F 2 "Package_TO_SOT_SMD:SOT-23" H 9100 1450 50  0001 C CNN
+F 3 "" H 9200 1200 50  0001 C CNN
+	1    9100 1450
+	1    0    0    -1
+$EndComp
+Wire Wire Line
+	7500 3400 7700 3400
+$Comp
+L Connector_Generic:Conn_01x01 J3
+U 1 1 622DF5F0
+P 4100 4250
+F 0 "J3" H 3950 4300 50  0000 L CNN
+F 1 "UART_TX" H 4200 4250 50  0000 L CNN
+F 2 "Connector_PinSocket_2.54mm:PinSocket_1x01_P2.54mm_Vertical" H 4100 4250 50  0001 C CNN
+F 3 "~" H 4100 4250 50  0001 C CNN
+	1    4100 4250
+	-1   0    0    1
+$EndComp
+$Comp
+L Connector_Generic:Conn_01x01 J4
+U 1 1 622E1A60
+P 4100 4350
+F 0 "J4" H 3950 4400 50  0000 L CNN
+F 1 "UART_RX" H 4200 4350 50  0000 L CNN
+F 2 "Connector_PinSocket_2.54mm:PinSocket_1x01_P2.54mm_Vertical" H 4100 4350 50  0001 C CNN
+F 3 "~" H 4100 4350 50  0001 C CNN
+	1    4100 4350
+	-1   0    0    1
+$EndComp
+Wire Wire Line
+	4300 4250 4500 4250
+Wire Wire Line
+	4500 4350 4300 4350
+$Comp
+L Connector_Generic:Conn_01x01 J5
+U 1 1 6230AF55
+P 4100 4450
+F 0 "J5" H 3950 4500 50  0000 L CNN
+F 1 "GND" H 4200 4450 50  0000 L CNN
+F 2 "Connector_PinSocket_2.54mm:PinSocket_1x01_P2.54mm_Vertical" H 4100 4450 50  0001 C CNN
+F 3 "~" H 4100 4450 50  0001 C CNN
+	1    4100 4450
+	-1   0    0    1
+$EndComp
+$Comp
+L power:GND #PWR0102
+U 1 1 6230BCA2
+P 4350 4500
+F 0 "#PWR0102" H 4350 4250 50  0001 C CNN
+F 1 "GND" H 4355 4327 50  0000 C CNN
+F 2 "" H 4350 4500 50  0001 C CNN
+F 3 "" H 4350 4500 50  0001 C CNN
+	1    4350 4500
+	1    0    0    -1
+$EndComp
+Wire Wire Line
+	4300 4450 4350 4450
+Wire Wire Line
+	4350 4450 4350 4500
 Wire Bus Line
 	3500 1350 3500 2700
@@
 Wire Bus Line
 	7850 1350 7850 3300
-Connection ~ 7700 3700
-Wire Wire Line
-	7700 3700 7800 3700
 $EndSCHEMATC
